File: pcbs/zapojeni-sonar/zapojeni-sonar.kicad_sch (KiCad schematic)
At the start: 4 parts, among them J1 Conn_01x20_Socket, J2 Conn_01x20_Socket, J3 Ultrazvukový senzor vzdálenos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, M1 Krokový motor 28BYJ-48

Commit message: t
Parts:
- added D1: RGB LED, symbol Device:LED_RGB
Connections:
- net GND: now also D1.1 (RK), D1.2 (GK), D1.3 (BK)
Other:
- note added: "BLUE"
- note added: "GREEN"
- note added: "RED"
Changed lines of the file:
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@@
 (kicad_sch (version 20230121) (generator eeschema)
   (paper "A4")
+  (junction (at 151.13 129.54) (diameter 0) (color 0 0 0 0)
+  )
   (junction (at 181.61 64.77) (diameter 0) (color 0 0 0 0)
   )
@@
   (junction (at 181.61 77.47) (diameter 0) (color 0 0 0 0)
   )
-  (wire (pts (xy 120.65 125.73) (xy 129.54 125.73))
+  (wire (pts (xy 124.46 95.25) (xy 142.24 95.25))
+    (stroke (width 0) (type default))
+  )
+  (wire (pts (xy 87.63 125.73) (xy 96.52 125.73))
     (stroke (width 0) (type default))
   )
@@
     (stroke (width 0) (type default))
   )
-  (wire (pts (xy 120.65 130.81) (xy 129.54 130.81))
+  (wire (pts (xy 163.83 134.62) (xy 172.72 134.62))
+    (stroke (width 0) (type default))
+  )
+  (wire (pts (xy 87.63 130.81) (xy 96.52 130.81))
     (stroke (width 0) (type default))
   )
@@
     (stroke (width 0) (type default))
   )
-  (wire (pts (xy 123.19 133.35) (xy 129.54 133.35))
+  (wire (pts (xy 153.67 134.62) (xy 151.13 134.62))
+    (stroke (width 0) (type default))
+  )
+  (wire (pts (xy 90.17 133.35) (xy 96.52 133.35))
     (stroke (width 0) (type default))
   )
@@
     (stroke (width 0) (type default))
   )
-  (wire (pts (xy 120.65 128.27) (xy 129.54 128.27))
+  (wire (pts (xy 151.13 134.62) (xy 151.13 129.54))
+    (stroke (width 0) (type default))
+  )
+  (wire (pts (xy 87.63 128.27) (xy 96.52 128.27))
     (stroke (width 0) (type default))
   )
@@
     (stroke (width 0) (type default))
   )
+  (wire (pts (xy 124.46 87.63) (xy 142.24 87.63))
+    (stroke (width 0) (type default))
+  )
   (wire (pts (xy 135.89 90.17) (xy 142.24 90.17))
     (stroke (width 0) (type default))
@@
     (stroke (width 0) (type default))
   )
+  (wire (pts (xy 151.13 124.46) (xy 153.67 124.46))
+    (stroke (width 0) (type default))
+  )
+  (wire (pts (xy 163.83 124.46) (xy 172.72 124.46))
+    (stroke (width 0) (type default))
+  )
+  (wire (pts (xy 147.32 129.54) (xy 151.13 129.54))
+    (stroke (width 0) (type default))
+  )
   (wire (pts (xy 175.26 64.77) (xy 181.61 64.77))
     (stroke (width 0) (type default))
@@
     (stroke (width 0) (type default))
   )
+  (wire (pts (xy 163.83 129.54) (xy 172.72 129.54))
+    (stroke (width 0) (type default))
+  )
   (wire (pts (xy 100.33 76.2) (xy 109.22 76.2))
     (stroke (width 0) (type default))
@@
     (stroke (width 0) (type default))
   )
+  (wire (pts (xy 151.13 129.54) (xy 151.13 124.46))
+    (stroke (width 0) (type default))
+  )
   (wire (pts (xy 181.61 77.47) (xy 181.61 64.77))
     (stroke (width 0) (type default))
@@
     (stroke (width 0) (type default))
   )
+  (wire (pts (xy 142.24 92.71) (xy 124.46 92.71))
+    (stroke (width 0) (type default))
+  )
   (wire (pts (xy 175.26 95.25) (xy 190.5 95.25))
     (stroke (width 0) (type default))
@@
     (stroke (width 0) (type default))
   )
+  (wire (pts (xy 151.13 129.54) (xy 153.67 129.54))
+    (stroke (width 0) (type default))
+  )
   (rectangle (start 80.01 69.85) (end 100.33 95.25)
     (stroke (width 0) (type default))
@@
     (fill (type none))
   )
-  (rectangle (start 134.62 121.92) (end 166.37 137.16)
+  (rectangle (start 101.6 121.92) (end 133.35 137.16)
     (stroke (width 0) (type default))
     (fill (type none))
   )
+  (text "GREEN" (at 124.46 92.71 0)
+    (effects (font (size 1.27 1.27)) (justify left bottom))
+  )
   (text "IN2\n" (at 109.22 76.2 0)
     (effects (font (size 1.27 1.27)) (justify right bottom))
@@
     (effects (font (size 1.27 1.27)) (justify right bottom))
   )
+  (text "RED" (at 124.46 87.63 0)
+    (effects (font (size 1.27 1.27)) (justify left bottom))
+  )
   (text "VBUS" (at 189.23 59.69 0)
     (effects (font (size 1.27 1.27)) (justify right bottom))
@@
     (effects (font (size 1.27 1.27)) (justify left bottom))
   )
-  (text "ECHO\n" (at 120.65 130.81 0)
+  (text "ECHO\n" (at 87.63 130.81 0)
     (effects (font (size 1.27 1.27)) (justify left bottom))
   )
@@
     (effects (font (size 1.27 1.27)) (justify left bottom))
   )
-  (text "VBUS\n" (at 120.65 125.73 0)
+  (text "VBUS\n" (at 87.63 125.73 0)
     (effects (font (size 1.27 1.27)) (justify left bottom))
   )
@@
     (effects (font (size 1.27 1.27)) (justify left bottom))
   )
+  (text "BLUE" (at 172.72 134.62 0)
+    (effects (font (size 1.27 1.27)) (justify right bottom))
+  )
   (text "Řadič ULN2003" (at 97.79 80.01 0)
     (effects (font (size 1.27 1.27)) (justify right bottom))
@@
     (effects (font (size 1.27 1.27)) (justify left bottom))
   )
-  (text "TRIGGER\n" (at 120.65 128.27 0)
+  (text "TRIGGER\n" (at 87.63 128.27 0)
     (effects (font (size 1.27 1.27)) (justify left bottom))
   )
@@
     (effects (font (size 1.27 1.27)) (justify right bottom))
   )
+  (text "GREEN" (at 172.72 129.54 0)
+    (effects (font (size 1.27 1.27)) (justify right bottom))
+  )
   (text "OUT3" (at 82.55 119.38 90)
     (effects (font (size 1.27 1.27)) (justify left bottom))
@@
     (effects (font (size 1.27 1.27)) (justify right bottom))
   )
+  (text "BLUE" (at 124.46 95.25 0)
+    (effects (font (size 1.27 1.27)) (justify left bottom))
+  )
   (text "OUT4" (at 71.12 86.36 0)
     (effects (font (size 1.27 1.27)) (justify left bottom))
+  )
+  (text "RED" (at 172.72 124.46 0)
+    (effects (font (size 1.27 1.27)) (justify right bottom))
   )
   (text "5V" (at 71.12 76.2 0)
@@
     )
   )
-  (symbol (lib_id "power:GND") (at 123.19 133.35 270) (unit 1)
+  (symbol (lib_id "power:GND") (at 147.32 129.54 270) (unit 1)
     (in_bom yes) (on_board yes) (dnp no) (fields_autoplaced)
-    (property "Reference" "#PWR03" (at 116.84 133.35 0)
-      (effects (font (size 1.27 1.27)) hide)
-    )
-    (property "Value" "GND" (at 119.38 133.35 90)
+    (property "Reference" "#PWR05" (at 140.97 129.54 0)
+      (effects (font (size 1.27 1.27)) hide)
+    )
+    (property "Value" "GND" (at 143.51 129.54 90)
       (effects (font (size 1.27 1.27)) (justify right))
     )
-    (property "Footprint" "" (at 123.19 133.35 0)
-      (effects (font (size 1.27 1.27)) hide)
-    )
-    (property "Datasheet" "" (at 123.19 133.35 0)
+    (property "Footprint" "" (at 147.32 129.54 0)
+      (effects (font (size 1.27 1.27)) hide)
+    )
+    (property "Datasheet" "" (at 147.32 129.54 0)
+      (effects (font (size 1.27 1.27)) hide)
+    )
+    (pin "1")
+    (instances
+      (project "zapojeni-sonar"
+        (path "/bf3bb856-b406-4ca1-810b-7f13d237ba92"
+          (reference "#PWR05") (unit 1)
+        )
+      )
+    )
+  )
+  (symbol (lib_id "power:GND") (at 90.17 133.35 270) (unit 1)
+    (in_bom yes) (on_board yes) (dnp no) (fields_autoplaced)
+    (property "Reference" "#PWR03" (at 83.82 133.35 0)
+      (effects (font (size 1.27 1.27)) hide)
+    )
+    (property "Value" "GND" (at 86.36 133.35 90)
+      (effects (font (size 1.27 1.27)) (justify right))
+    )
+    (property "Footprint" "" (at 90.17 133.35 0)
+      (effects (font (size 1.27 1.27)) hide)
+    )
+    (property "Datasheet" "" (at 90.17 133.35 0)
       (effects (font (size 1.27 1.27)) hide)
     )
@@
     )
   )
-  (symbol (lib_id "Connector:Conn_01x04_Socket") (at 134.62 128.27 0) (unit 1)
+  (symbol (lib_id "Connector:Conn_01x04_Socket") (at 101.6 128.27 0) (unit 1)
     (in_bom yes) (on_board yes) (dnp no)
-    (property "Reference" "J3" (at 135.89 128.27 0)
+    (property "Reference" "J3" (at 102.87 128.27 0)
       (effects (font (size 1.27 1.27)) (justify left) hide)
     )
-    (property "Value" "Ultrazvukový senzor vzdálenosti\n HC-SR04" (at 134.62 129.54 0)
+    (property "Value" "Ultrazvukový senzor vzdálenosti\n HC-SR04" (at 101.6 129.54 0)
       (effects (font (size 1.27 1.27)) (justify left))
     )
-    (property "Footprint" "" (at 134.62 128.27 0)
-      (effects (font (size 1.27 1.27)) hide)
-    )
-    (property "Datasheet" "~" (at 134.62 128.27 0)
+    (property "Footprint" "" (at 101.6 128.27 0)
+      (effects (font (size 1.27 1.27)) hide)
+    )
+    (property "Datasheet" "~" (at 101.6 128.27 0)
       (effects (font (size 1.27 1.27)) hide)
     )
@@
         )
       )
+    )
+  )
+  (symbol (lib_id "Device:LED_RGB") (at 158.75 129.54 0) (unit 1)
+    (in_bom yes) (on_board yes) (dnp no) (fields_autoplaced)
+    (property "Reference" "D1" (at 158.75 116.84 0)
+      (effects (font (size 1.27 1.27)) hide)
+    )
+    (property "Value" "RGB LED" (at 158.75 119.38 0)
+      (effects (font (size 1.27 1.27)))
+    )
+    (property "Footprint" "" (at 158.75 130.81 0)
+      (effects (font (size 1.27 1.27)) hide)
+    )
+    (property "Datasheet" "~" (at 158.75 130.81 0)
+      (effects (font (size 1.27 1.27)) hide)
+    )
+    (pin "1")
+    (pin "2")
+    (pin "3")
+    (pin "4")
+    (pin "5")
+    (pin "6")
+    (instances
+      (project "zapojeni-sonar"
+        (path "/bf3bb856-b406-4ca1-810b-7f13d237ba92"
+          (reference "D1") (unit 1)
+        )
+      )

Commit message: AYOOO
Connections:
- net GND: now also J1.16 (Pin_16)
Other:
- note added: "Příloha VII: Schéma zapojení součástek"
- note added: "UART0 RX"
- note added: "UART0 TX"
- title: (none) -> Schéma zapojení součástek
